Commit message: summarize sensor xacro

File: whill_sensor_kit_description/urdf/sensors.xacro (robot description, xacro)
@@ -3,14 +3,16 @@
   <xacro:arg name="config_dir" default="$(find whill_sensor_kit_description)/config"/>
   <xacro:property name="calibration" value="${xacro.load_yaml('$(arg config_dir)/sensors_calibration.yaml')}"/>
-  <!-- sensor kit -->
-  <xacro:include filename="sensor_kit.xacro"/>
-  <xacro:sensor_kit_macro
-    parent="base_link"
-    x="${calibration['base_link']['sensor_kit_base_link']['x']}"
-    y="${calibration['base_link']['sensor_kit_base_link']['y']}"
-    z="${calibration['base_link']['sensor_kit_base_link']['z']}"
-    roll="${calibration['base_link']['sensor_kit_base_link']['roll']}"
-    pitch="${calibration['base_link']['sensor_kit_base_link']['pitch']}"
-    yaw="${calibration['base_link']['sensor_kit_base_link']['yaw']}"
-  />
+  <xacro:include filename="$(find velodyne_description)/urdf/VLP-16.urdf.xacro"/>
+  <xacro:arg name="gpu" default="false"/>
+  <!-- lidar -->
+  <xacro:VLP-16 parent="base_link" name="velodyne_top" topic="/points_raw" hz="10" samples="220" gpu="$(arg gpu)">
+    <origin
+      xyz="${calibration['base_link']['velodyne_top_base_link']['x']}
+            ${calibration['base_link']['velodyne_top_base_link']['y']}
+            ${calibration['base_link']['velodyne_top_base_link']['z']}"
+      rpy="${calibration['base_link']['velodyne_top_base_link']['roll']}
+            ${calibration['base_link']['velodyne_top_base_link']['pitch']}
+            ${calibration['base_link']['velodyne_top_base_link']['yaw']}"
+    />
+  </xacro:VLP-16>
 </robot>
